File: PCB/WSB-PC/WSB-PC.kicad_pcb (KiCad board)
At the start: 6 copper layers, 16 x 15 mm, 35 parts, among them P1 GT-USB-8012A, SW1 SW_SPST_4_PIN, U1 74LV1T34, U2 ESP32-C6-MINI-1, U4 TPD2E2U06DRL, U5 NCP187

Commit message: -Corrected test point numbering
Parts:
- renumbered C30 to C1, C23 to C10, C31 to C2, C35 to C3, C1 to C4, C2 to C5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
