File: PCB/WSB-PC/.history/WSB-PC.kicad_sch (KiCad schematic)
At the start: 34 parts, among them P2 USB_C_Plug_USB2.0, SW1 SW_SPST_4_PIN, U1 ESP32-C6-MINI-1, U2 74LV1T34, U3 NCP187, U4 TPD2E2U06DRL

Commit message: -Changed USB connector -Moved LEDs in behind board edge -Changed to smaller test points
Parts:
- TP1, TP2, TP3, TP4, TP5, TP6, TP7, TP8: footprint EN_Designs-Footprints:TestPoint_Pad_D0.5mm -> EN_Designs-Footprints:TestPoint_Pad_D1.0mm
- U2: footprint EN_Designs-Footprints:X2SON5_0.8x0.8mm_SOT1226 -> EN_Designs-KiCad-Lib:X2SON5_0.8x0.8mm_SOT1226
Changed lines of the file:
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@@
 			)
 		)
-		(property "Footprint" "EN_Designs-Footprints:TestPoint_Pad_D0.5mm"
+		(property "Footprint" "EN_Designs-Footprints:TestPoint_Pad_D1.0mm"
 			(at 115.57 45.72 0)
 			(hide yes)
@@
 			)
 		)
-		(property "Footprint" "EN_Designs-Footprints:X2SON5_0.8x0.8mm_SOT1226"
+		(property "Footprint" "EN_Designs-KiCad-Lib:X2SON5_0.8x0.8mm_SOT1226"
 			(at 165.1 72.39 0)
 			(hide yes)
@@
 			)
 		)
-		(property "Footprint" "EN_Designs-Footprints:TestPoint_Pad_D0.5mm"
+		(property "Footprint" "EN_Designs-Footprints:TestPoint_Pad_D1.0mm"
 			(at 85.09 121.92 0)
 			(hide yes)
@@
 			)
 		)
-		(property "Footprint" "EN_Designs-Footprints:TestPoint_Pad_D0.5mm"
+		(property "Footprint" "EN_Designs-Footprints:TestPoint_Pad_D1.0mm"
 			(at 153.67 71.12 0)
 			(hide yes)
@@
 			)
 		)
-		(property "Footprint" "EN_Designs-Footprints:TestPoint_Pad_D0.5mm"
+		(property "Footprint" "EN_Designs-Footprints:TestPoint_Pad_D1.0mm"
 			(at 144.78 121.92 0)
 			(hide yes)
@@
 			)
 		)
-		(property "Footprint" "EN_Designs-Footprints:TestPoint_Pad_D0.5mm"
+		(property "Footprint" "EN_Designs-Footprints:TestPoint_Pad_D1.0mm"
 			(at 67.31 160.02 0)
 			(hide yes)
@@
 			)
 		)
-		(property "Footprint" "EN_Designs-Footprints:TestPoint_Pad_D0.5mm"
+		(property "Footprint" "EN_Designs-Footprints:TestPoint_Pad_D1.0mm"
 			(at 62.23 74.93 0)
 			(hide yes)
@@
 			)
 		)
-		(property "Footprint" "EN_Designs-Footprints:TestPoint_Pad_D0.5mm"
+		(property "Footprint" "EN_Designs-Footprints:TestPoint_Pad_D1.0mm"
 			(at 109.22 45.72 0)
 			(hide yes)
@@
 			)
 		)
-		(property "Footprint" "EN_Designs-Footprints:TestPoint_Pad_D0.5mm"
+		(property "Footprint" "EN_Designs-Footprints:TestPoint_Pad_D1.0mm"
 			(at 62.23 46.99 0)
 			(hide yes)
